File: HARP-Motor-Ctrl-Board/HARP-Motor-Ctrl-Board.kicad_pcb (KiCad board)
At the start: 2 copper layers, 30 x 59 mm, 21 parts, among them IC1 TC7S14F,LF, IC2 TC7S14F,LF, IC3 STM32L010F4P6, IC4 TC7S14F,LF, IC5 TC7S14F,LF, J1 Conn_01x05_Male, J2 Conn_01x04_Male, J3 Conn_01x02_Male, J4 Conn_01x05_Male, J5 Conn_01x05_Male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

Commit message: added logo and regenerated gerber files.
Parts:
- removed the REF** at (88.0, 97.0)
Other:
- board text added: "Project HARP Motor Ctrl Brd 1.0 Designed by Soula."
